File: shell/快速结构预览/pcb/preview-local-mount.kicad_pcb (KiCad board)
At the start: 2 copper layers, 52 x 82 mm, 24 parts, among them SW1 HW-504 34x26mm, SW1_ALT HW-504直排针备用位, SW2 D2FC-F-7N(20M)

Commit message: 移除上部框架并重排电源开关和惯性模块固定孔
Parts:
- added H_BODY_5: , , F.Cu at (40.5, 83.0)
- added H_IMU_1: , , F.Cu at (50.8, 28.6)
- added H_IMU_2: , , F.Cu at (50.8, 13.4)
- moved J_SWITCH 43.8 mm to (50.0, 41.0)
- moved J_GY 2.20 mm to (47.1, 20.8)
Routing:
- net BAT_RAW: track 10.5 -> 40.9 mm
- net BAT_SW: track 98.1 -> 90.5 mm
- net 3V3: track 70.7 -> 77.0 mm, vias 0 -> 2
- net JOY_SW: track 150.7 -> 155.1 mm
- net GND: track 171.0 -> 174.1 mm
- net SCL: track 34.3 -> 37.4 mm
- net SDA: track 19.9 -> 18.8 mm
